File: KiCAD/microbit-enviromonitor-board/microbit-enviromonitor-board.sch (KiCad schematic (older format))
At the start: 8 parts, among them J1 12V, J2 SERIAL, J3 3V3, J4 PUMP, Q1 TIP41C, U1 REGULATOR

Commit message: Updated serial port
Parts:
- removed J2: SERIAL, headers:2_double_spaced, symbol Connector:Screw_Terminal_01x02
- added J2: SERIAL, headers:4x1, symbol Connector:Conn_01x04_Female
- U1: footprint headers:4x1 -> misc:buck_converter
Connections:
- net +3V3: now also J2.3 (Pin_3)
- net GND: now also J2.4 (Pin_4)
- net at E1.12 (RX0): now also J2.2 (Pin_2)
- net at E1.13 (TX0): now also J2.1 (Pin_1)
Changed lines of the file:
@@
 F 0 "U1" H 2400 1815 50  0000 C CNN
 F 1 "REGULATOR" H 2400 1724 50  0000 C CNN
-F 2 "headers:4x1" H 2400 1550 50  0001 C CNN
+F 2 "misc:buck_converter" H 2400 1550 50  0001 C CNN
 F 3 "" H 2400 1550 50  0001 C CNN
 	1    2400 1550
@@
 Text Label 2700 2900 0    50   ~ 0
 PUMP
-$Comp
-L Connector:Screw_Terminal_01x02 J2
-U 1 1 5F0D99D4
-P 2950 3100
-F 0 "J2" H 3030 3092 50  0000 L CNN
-F 1 "SERIAL" H 3030 3001 50  0000 L CNN
-F 2 "headers:2_double_spaced" H 2950 3100 50  0001 C CNN
-F 3 "~" H 2950 3100 50  0001 C CNN
-	1    2950 3100
-	1    0    0    -1
-$EndComp
-Wire Wire Line
-	2750 3100 2600 3100
-Wire Wire Line
-	2750 3200 2600 3200
 Wire Notes Line
 	1400 2500 1400 4750
@@
 Text Notes 3200 2450 0    50   ~ 0
 ESP32
+$Comp
+L Connector:Conn_01x04_Female J2
+U 1 1 5F10408E
+P 3150 3200
+F 0 "J2" H 3178 3176 50  0000 L CNN
+F 1 "SERIAL" H 3178 3085 50  0000 L CNN
+F 2 "headers:4x1" H 3150 3200 50  0001 C CNN
+F 3 "~" H 3150 3200 50  0001 C CNN
+	1    3150 3200
+	1    0    0    -1
+$EndComp
+Wire Wire Line
+	2600 3100 2950 3100
+Wire Wire Line
+	2600 3200 2950 3200
+$Comp
+L power:GND #PWR02
+U 1 1 5F10692A
+P 2800 3500
+F 0 "#PWR02" H 2800 3250 50  0001 C CNN
+F 1 "GND" H 2805 3327 50  0000 C CNN
+F 2 "" H 2800 3500 50  0001 C CNN
+F 3 "" H 2800 3500 50  0001 C CNN
+	1    2800 3500
+	1    0    0    -1
+$EndComp
+$Comp
+L power:+3V3 #PWR01
+U 1 1 5F107157
+P 2800 3050
+F 0 "#PWR01" H 2800 2900 50  0001 C CNN
+F 1 "+3V3" H 2950 3150 50  0000 C CNN
+F 2 "" H 2800 3050 50  0001 C CNN
+F 3 "" H 2800 3050 50  0001 C CNN
+	1    2800 3050
+	1    0    0    -1
+$EndComp
+Wire Wire Line
+	2800 3050 2800 3300
+Wire Wire Line
+	2800 3300 2950 3300
+Wire Wire Line
+	2800 3500 2800 3400
+Wire Wire Line
+	2800 3400 2950 3400
 $EndSCHEMATC

Commit message: Board changes
Parts:
- J1, J3, J4: footprint headers:2_double_spaced -> headers:screw_terminal
Changed lines of the file:
@@
 F 0 "J1" H 1468 1325 50  0000 C CNN
 F 1 "12V" H 1468 1416 50  0000 C CNN
-F 2 "headers:2_double_spaced" H 1550 1650 50  0001 C CNN
+F 2 "headers:screw_terminal" H 1550 1650 50  0001 C CNN
 F 3 "~" H 1550 1650 50  0001 C CNN
 	1    1550 1650
@@
 F 0 "J4" H 4930 1292 50  0000 L CNN
 F 1 "PUMP" H 4930 1201 50  0000 L CNN
-F 2 "headers:2_double_spaced" H 4850 1300 50  0001 C CNN
+F 2 "headers:screw_terminal" H 4850 1300 50  0001 C CNN
 F 3 "~" H 4850 1300 50  0001 C CNN
 	1    4850 1300
@@
 F 0 "J3" H 3280 1542 50  0000 L CNN
 F 1 "3V3" H 3280 1451 50  0000 L CNN
-F 2 "headers:2_double_spaced" H 3200 1550 50  0001 C CNN
+F 2 "headers:screw_terminal" H 3200 1550 50  0001 C CNN
 F 3 "~" H 3200 1550 50  0001 C CNN
 	1    3200 1550

Commit message: Added pump switch
Connections:
- net at E1.12 (RX0): no longer J2.2 (Pin_2)
- net at E1.13 (TX0): no longer J2.1 (Pin_1)
- net at E1.6 (RX2): now also J2.2 (Pin_2)
- net at E1.7 (TX2): now also J2.1 (Pin_1)
Changed lines of the file:
@@
 	1    0    0    -1
 $EndComp
-Wire Wire Line
-	2600 3100 2950 3100
-Wire Wire Line
-	2600 3200 2950 3200
 $Comp
 L power:GND #PWR02
@@
 Wire Wire Line
 	2800 3400 2950 3400
+Wire Wire Line
+	2950 3100 2650 3100
+Wire Wire Line
+	2650 3100 2650 3700
+Wire Wire Line
+	2650 3700 2600 3700
+Wire Wire Line
+	2950 3200 2700 3200
+Wire Wire Line
+	2700 3200 2700 3800
+Wire Wire Line
+	2700 3800 2600 3800
 $EndSCHEMATC
